File: Phobri64/Phobri64.kicad_pcb (KiCad board)
At the start: 2 copper layers, 99.5 x 69.4 mm, 176 parts, among them J12 Mobo_To_Stick, J2 HoriStyleStick, J3 Conn_01x03, J4 L_Board, J5 R_Board, J6 N64_Intf, J7 Stick_To_Mobo, J8 USB_C_Receptacle, J9 Conn_01x03, SW1 A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

Commit message: The stick-box now fits even if its structural pins are rotated
Parts:
- moved R5 1.62 mm to (163.4, 101.7), turned to -45 degrees
- moved C4 0.51 mm to (166.7, 96.6)
- moved TVS_19 0.51 mm to (161.8, 100.3)
- moved C6 0.51 mm to (165.6, 95.5)
- moved U2 0.51 mm to (163.7, 98.3)
- moved TP5 0.13 mm to (160.7, 95.9)
Routing:
- net S_GND: track 246.9 -> 251.6 mm, vias 85 -> 91
- net +S_3V3: track 74.3 -> 77.7 mm
- net Net-(U2-ALERT_N): track 1.60 -> 2.47 mm
- net /POT_X: track 14.5 -> 15.0 mm
